File: .history/BT.kicad_sch (KiCad schematic)
At the start: 95 parts, among them J1 61300511121, J2 S3B-PH-K-S, J3 S6B-PH-K-S, J4 Boxed_Header_02x03_SMT, K1 AGQ200A12Z, M1 Mounting_Hole_2.7mm_Unplated, M2 Mounting_Hole_2.7mm_Unplated, M3 Mounting_Hole_2.7mm_Unplated, Q1 BSS123, U1 PCM5100A, U2 ESP32-WROOM-32U, U3 TLV4888DR, U4 TLVM23615RDNR, U5 TLVM23615RDNR, U6 RAA214220, Y1 XO32

Commit message: almost finished layout. Something is still off in the design rules
Connections:
- net +3.3VA is gone; now on net +3V3A: C3.1, C4.1, U1.8 (AVDD)
- net DAC_FLT: now also U2.30 (IO18); no longer U2.33 (IO21)
- net DAC_FMT: now also U2.33 (IO21); no longer U2.10 (IO25)
Changed lines of the file:
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@@
 	)
 	(no_connect
-		(at 93.98 99.06)
-	)
-	(no_connect
 		(at 257.81 242.57)
 	)
@@
 	)
 	(no_connect
+		(at 93.98 111.76)
+	)
+	(no_connect
 		(at 93.98 73.66)
 	)
@@
 	(wire
 		(pts
-			(xy 93.98 104.14) (xy 144.78 104.14)
+			(xy 93.98 104.14) (xy 152.4 104.14)
 		)
 		(stroke
@@
 	(wire
 		(pts
-			(xy 152.4 72.39) (xy 152.4 111.76)
+			(xy 152.4 72.39) (xy 152.4 104.14)
 		)
 		(stroke
@@
 	(wire
 		(pts
+			(xy 144.78 64.77) (xy 144.78 99.06)
+		)
+		(stroke
+			(width 0)
+			(type default)
+		)
+	)
+	(wire
+		(pts
 			(xy 346.71 62.23) (xy 368.3 62.23)
 		)
@@
 	(wire
 		(pts
+			(xy 93.98 99.06) (xy 144.78 99.06)
+		)
+		(stroke
+			(width 0)
+			(type default)
+		)
+	)
+	(wire
+		(pts
 			(xy 170.18 116.84) (xy 170.18 127)
 		)
@@
 	(wire
 		(pts
-			(xy 93.98 111.76) (xy 152.4 111.76)
-		)
-		(stroke
-			(width 0)
-			(type default)
-		)
-	)
-	(wire
-		(pts
 			(xy 157.48 81.28) (xy 157.48 91.44)
 		)
@@
 	(wire
 		(pts
-			(xy 144.78 64.77) (xy 144.78 104.14)
-		)
-		(stroke
-			(width 0)
-			(type default)
-		)
-	)
-	(wire
-		(pts
 			(xy 22.86 21.59) (xy 22.86 27.94)
 		)
@@
 		)
 	)
-	(label "DAC_FLT"
+	(label "DAC_FMT"
 		(at 113.03 104.14 180)
 		(effects
@@
 		)
 	)
-	(label "DAC_FMT"
-		(at 113.03 111.76 180)
-		(effects
-			(font
-				(size 1.27 1.27)
-			)
-			(justify right bottom)
-		)
-	)
 	(label "ESP_IO0"
 		(at 55.88 210.82 180)
@@
 		)
 	)
+	(label "DAC_FLT"
+		(at 113.03 99.06 180)
+		(effects
+			(font
+				(size 1.27 1.27)
+			)
+			(justify right bottom)
+		)
+	)
 	(label "BCK"
 		(at 139.7 57.15 0)
@@
 			)
 		)
-		(property "Value" "+3.3VA"
+		(property "Value" "+3V3A"
 			(at 157.226 18.034 0)
 			(show_name no)
