File: BT.kicad_pcb (KiCad board)
At the start: 4 copper layers, 55 x 40 mm, 97 parts, among them J1 61300511121, J2 S6B-PH-K-S, J3 S6B-PH-K-S, J4 Boxed_Header_02x03_SMT, K1 AGQ200A12Z, M1 Mounting_Hole_2.7mm_Unplated, M2 Mounting_Hole_2.7mm_Unplated, M3 Mounting_Hole_2.7mm_Unplated, Q1 BSS123, Q2 BSS123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

Commit message: Release Rev. A
Parts:
- moved R13 3.85 mm to (126.5, 87.0), turned to 90 degrees
- moved J1 3.07 mm to (132.8, 90.9)
- moved TP3 0.95 mm to (159.0, 95.2)
- moved TP2 0.90 mm to (164.9, 95.2)
- moved M3 0.46 mm to (172.7, 112.7)
Connections:
- U2 pad 11: /DAC_MCLK_EN -> /BT_EN
- U2 pad 6: /BT_EN -> /DAC_MCLK_EN
Routing:
- net /MCLK: track 12.1 -> 21.0 mm
- net /KL30: track 19.1 -> 15.0 mm
- net /DAC_FLT: track 13.3 -> 9.21 mm
- net /DAC_MCLK_EN: track 33.8 -> 29.9 mm
- net /DAC_MUTEn: track 23.3 -> 20.3 mm
- net /LED: track 39.1 -> 41.8 mm
- net /REV_CON: track 47.5 -> 50.1 mm
- net GND: track 68.1 -> 70.5 mm, vias 60 -> 79
- net /BCK: track 9.72 -> 12.1 mm
- net /LRCK: track 10.5 -> 8.58 mm
- net +3V3: track 35.4 -> 37.2 mm
- net /ESP_RXD0: track 32.7 -> 34.4 mm
- net /DIN: track 8.79 -> 10.3 mm
- net /FWD_CON: track 40.8 -> 42.3 mm
- net /SCK: track 17.6 -> 18.6 mm
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Other:
- board text added: "BT Alpha Rev. A"
- board text added: "BT_EN"
- board text added: "FWD_CON"
- board text added: "GND"
- board text added: "KL30"
- board text added: "LED_CON"
- board text added: "L_IN"
- board text added: "L_OUT"
- board text added: "REV_CON"
- board text added: "R_IN"
- board text added: "R_OUT"
- board text added: "~{BT_EN}"
