File: BT.kicad_sch (KiCad schematic)
At the start: 95 parts, among them J1 61300511121, J2 S3B-PH-K-S, J3 S6B-PH-K-S, J4 Boxed_Header_02x03_SMT, K1 AGQ200A12Z, M1 Mounting_Hole_2.7mm_Unplated, M2 Mounting_Hole_2.7mm_Unplated, M3 Mounting_Hole_2.7mm_Unplated, Q1 BSS123, U1 PCM5100A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

Commit message: added signals
Parts:
- removed C22: 100nF, NRD_CAP:C_0603, symbol NRD_C_0603:CL10B104KB8NNNC
- removed J2: S3B-PH-K-S, NRD_CON:S3B-PH-K-S, symbol NRD_CON:S3B-PH-K-S
- removed R35, R6: 1K, NRD_RES:R_0603, symbol NRD_R_0603:RC0603FR-071KL
- removed R7: 10K, NRD_RES:R_0603, symbol NRD_R_0603:RC0603FR-0710KL
- added C28, C34: 100nF, NRD_CAP:C_0603, symbol NRD_C_0603:CL10B104KB8NNNC
- added J2: S6B-PH-K-S, NRD_CON:S6B-PH-K-S, symbol NRD_CON:S6B-PH-K-S
- added Q2: BSS123, NRD_MOSFET:BSS123, symbol NRD_MOSFET:BSS123
- added R38, R39: 10K, NRD_RES:R_0603, symbol NRD_R_0603:RC0603FR-0710KL
- added R40: 1K, NRD_RES:R_0603, symbol NRD_R_0603:RC0603FR-071KL
- D1: Manufacturer Visha -> Vishay
Connections:
- net +3V3: now also R34.1, R38.2, R39.2
- net DAC_MCLK_EN: now also U2.11 (IO26); no longer U2.8 (IO32)
- net DAC_MUTEn: no longer R34.1
- net GND: now also C28.2, C34.2, J2.1 (Pin_1), Q2.2 (S); no longer R34.2
- net LED: now also U2.9 (IO33), R40.2; no longer U2.11 (IO26)
- net LED_CON: now also J2.5 (Pin_5), R40.1
- net BT_EN: now reaches U2.6 (IO34)
- net BT_EN: now also Q1.1 (G), R8.1, J2.6 (Pin_6), Q2.1 (G)
- net Button renamed FWD_CON
- net FWD_CON: now also C28.1, J2.3 (Pin_3), R38.1
- removed net SW_TO_BT_AUDIO: Q1.1 (G), R8.1, U2.7 (IO35)
- new net REV_CON: C34.1, J2.4 (Pin_4), R39.1, U2.8 (IO32)
- new net ~{BT_EN}: J2.2 (Pin_2), Q2.3 (D), R34.2
- no-connect marks 28 -> 27
Other:
- note added: "BT_EN"
- note added: "LED: Kingbright WP710A10QBC/D"
- note added: "Pole Switch_ C&K 7105SYZQE"
- moved on the sheet: C16, C8, C9, R1, R13, R14, R15, R16, R8, Y1

Commit message: Release Rev. A
Connections:
- net BT_EN: now also U2.11 (IO26); no longer U2.6 (IO34)
- net DAC_MCLK_EN: now also U2.6 (IO34); no longer U2.11 (IO26)
Other:
- note added: "credits amplifier: https://electronics.stackexchange.com/questions/450609/op-amp-circuit-to-control-gain-of-two-analog-channels-with-one-single-section-po"
- note added: "swiching left short: revert track switching left long: toggle between normal radio and bluetooth switching right short: forward track switching right long: paring mode"
- note removed: "credits: https://electronics.stackexchange.com/questions/450609/op-amp-circuit-to-control-gain-of-two-analog-channels-with-one-single-section-po"
- moved on the sheet: C27, C28, C34, C35, C36, L1, L2, R38, R39, R40, U3D, U3E
