File: BT_Alpha.kicad_sch (KiCad schematic)
At the start: 97 parts, among them J1 61300511121, J2 S6B-PH-K-S, J3 S6B-PH-K-S, J4 Boxed_Header_02x03_SMT, K1 AGQ200A12Z, M1 Mounting_Hole_2.7mm_Unplated, M2 Mounting_Hole_2.7mm_Unplated, M3 Mounting_Hole_2.7mm_Unplated, Q1 BSS123, Q2 BSS123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

Commit message: renamed project
Other:
- company: Pfusch & Murks AG -> (none)
- title: 6B - BangBoomBlauzahnBlaupunktBassBox -> BT_Alpha
