File: BT_Alpha.kicad_pcb (KiCad board)
At the start: 4 copper layers, 55 x 40 mm, 97 parts, among them J1 61300511121, J2 S6B-PH-K-S, J3 S6B-PH-K-S, J4 Boxed_Header_02x03_SMT, K1 AGQ200A12Z, M1 Mounting_Hole_2.7mm_Unplated, M2 Mounting_Hole_2.7mm_Unplated, M3 Mounting_Hole_2.7mm_Unplated, Q1 BSS123, Q2 BSS123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

Commit message: started iterating to rev. B
Parts:
- removed C16: 100nF, NRD_CAP:C_0603
- removed C8, C9: 3.3nF, NRD_CAP:C_0603
- removed J1: 61300511121, NRD_PinHeader:61300511121
- removed R1, R4: 470R, NRD_RES:R_0603
- removed R10, R11, R12, R22, R23, R24, R25, R27, R28, R29, R30, R9: 1M, NRD_RES:R_0603
- removed R13, R14, R15: 0R, NRD_RES:R_0603
- removed R16, R21, R26: 10K, NRD_RES:R_0603
- removed R33: 10K, NRD_R_Var:TC33X-2
- removed Y1: XO32, Oscillator:Oscillator_SMD_EuroQuartz_XO32-4Pin_3.2x2.5mm
- added C22: 10uF, NRD_CAP:C_0805, F.Cu at (143.2, 81.0)
- added C37: 10uF, NRD_CAP:C_0805, F.Cu at (143.2, 83.0)
- added R41: 10K, NRD_RES:R_0603, F.Cu at (146.4, 85.4)
- added R42: 10K, NRD_RES:R_0603, F.Cu at (146.4, 80.9)
- added R43: 10K, NRD_RES:R_0603, F.Cu at (146.4, 83.9)
- added R44: 10K, NRD_RES:R_0603, F.Cu at (146.4, 82.4)
- U3: value TLV4888DR -> TLV2888DR; footprint NRD_IC_OPAMP:TLV4888DR -> NRD_IC_OPAMP:TLV2888DR
- moved TP1 17.7 mm to (155.7, 77.7)
- moved TP2 16.2 mm to (155.7, 81.9)
- moved C14 12.8 mm to (155.7, 84.7)
- moved R8 10.3 mm to (169.4, 78.1), turned to 90 degrees
- moved C27 7.80 mm to (152.9, 89.6), turned to 90 degrees
- moved C15 6.69 mm to (155.8, 87.3)
- moved TP3 5.97 mm to (155.9, 90.1)
- moved C36 5.36 mm to (151.2, 89.6), turned to 90 degrees
- moved Q1 5.30 mm to (166.9, 78.2), turned to 180 degrees
- moved D1 4.66 mm to (161.9, 78.2), turned to 0 degrees
- moved R32 3.29 mm to (128.6, 86.0)
- moved L2 2.53 mm to (149.2, 89.6), turned to -90 degrees
- moved L1 2.43 mm to (145.7, 89.6), turned to 90 degrees
- moved U3 1.67 mm to (151.1, 84.1), turned to -90 degrees
- moved K1 0.65 mm to (162.2, 85.8)
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Connections:
- C14 pad 2: Net-(C14-Pad2) -> Net-(U3A--)
- C15 pad 2: Net-(C15-Pad2) -> Net-(U3B--)
- C27 pad 1: Net-(U3E-V+) -> +6V_FLT
- C36 pad 1: Net-(U3E-V+) -> +6V_FLT
- K1 pad 1: +12V -> Net-(Q1-D)
- K1 pad 8: Net-(Q1-D) -> +12V
- L2 pad 2: Net-(U3E-V+) -> +6V_FLT
- TP2 pad 1: Net-(C14-Pad2) -> Net-(U3A--)
- TP3 pad 1: Net-(C15-Pad2) -> Net-(U3B--)
- U1 pad 12: /SCK -> /ESP_IO0
- U2 pad 27: /MCLK -> unconnected-(U2-IO16-Pad27)
- U3 pad 1: Net-(R10-Pad1) -> Net-(U3A--)
- U3 pad 4: Net-(U3E-V+) -> GND
- U3 pad 7: Net-(R24-Pad1) -> Net-(U3B--)
- U3 pad 8: Net-(C15-Pad2) -> +6V_FLT
Routing:
- net Net-(C14-Pad2): track 41.4 -> 0.00 mm, vias 2 -> 0
- net /ESP_IO0: track 18.9 -> 44.4 mm, vias 0 -> 2
- net /MCLK: track 21.0 -> 0.00 mm, vias 2 -> 0
- net Net-(C8-Pad1): track 19.4 -> 0.00 mm, vias 2 -> 0
- net Net-(R25-Pad1): track 18.6 -> 0.00 mm, vias 2 -> 0
- net /BT_EN: track 127.7 -> 109.1 mm, vias 3 -> 2
- net /SCK: track 18.6 -> 0.00 mm, vias 2 -> 0
- net Net-(R24-Pad1): track 17.4 -> 0.00 mm, vias 2 -> 0
- net Net-(U3B-+): track 15.9 -> 0.00 mm, vias 2 -> 0
- net Net-(U3C-+): track 10.6 -> 0.00 mm
- net GND: track 70.5 -> 60.3 mm, vias 79 -> 60
- net Net-(C15-Pad2): track 9.69 -> 0.00 mm
- net Net-(R10-Pad1): track 6.69 -> 0.00 mm
- net Net-(U3E-V+): track 6.63 -> 0.00 mm
- net Net-(U3A--): track 5.83 -> 0.00 mm
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- added copper zone on F.Cu, net (none)
- removed copper zone on F.Cu, net +3V3A
Other:
- board text added: "BT Alpha Rev. B"
- board text removed: "BT Alpha Rev. A"

Commit message: wip
Parts:
- removed TP1, TP2, TP3: 5001, NRD_MISC:500x
- moved U3 0.90 mm to (151.1, 83.2)

Commit message: added credits
Routing:
- net +12V: track 37.5 -> 31.1 mm, vias 1 -> 2
- net GND: vias 60 -> 59
Changed lines of the file:
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@@
-	)
-	(via
-		(at 158.09 81.01)
-		(size 0.6)
-		(drill 0.3)
-		(layers "F.Cu" "B.Cu")
-		(net "GND")
 	)
 	(via
@@
 	)
 	(via
-		(at 158.615 103.835)
+		(at 158.29 103.91)
 		(size 0.6)
 		(drill 0.3)
@@
 		(net "+12V")
 	)
-	(segment
-		(start 171.815 83.31)
-		(end 168.665 80.16)
+	(via
+		(at 158.29 78.21)
+		(size 0.6)
+		(drill 0.3)
+		(layers "F.Cu" "B.Cu")
+		(net "+12V")
+	)
+	(segment
+		(start 158.29 103.91)
+		(end 158.29 78.21)
 		(width 0.4)
 		(layer "In1.Cu")
@@
 	)
 	(segment
-		(start 161.465 103.835)
-		(end 171.815 93.485)
-		(width 0.4)
-		(layer "In1.Cu")
-		(net "+12V")
-	)
-	(segment
-		(start 171.815 93.485)
-		(end 171.815 83.31)
-		(width 0.4)
-		(layer "In1.Cu")
-		(net "+12V")
-	)
-	(segment
-		(start 158.615 103.835)
-		(end 161.465 103.835)
-		(width 0.4)
-		(layer "In1.Cu")
-		(net "+12V")
-	)
-	(segment
 		(start 135.69 88.01)
 		(end 135.69 86.135)
@@
 	(segment
 		(start 148.19 93.185)
-		(end 157.915 102.91)
+		(end 157.39 102.385)
 		(width 0.5)
 		(layer "In2.Cu")
@@
 	)
 	(segment
-		(start 157.915 108.735)
+		(start 157.39 102.385)
+		(end 157.39 108.21)
+		(width 0.5)
+		(layer "In2.Cu")
+		(net "+6V")
+	)
+	(segment
+		(start 157.39 108.21)
 		(end 162.74 113.56)
 		(width 0.5)
 		(layer "In2.Cu")
-		(net "+6V")
-	)
-	(segment
-		(start 157.915 102.91)
-		(end 157.915 108.735)
-		(width 0.5)
-		(layer "In2.Cu")

Commit message: diameter
Parts:
- M1, M2, M3: value Mounting_Hole_2.7mm_Unplated -> Val**
